File: electronics/STImu.kicad_pcb (KiCad board)
At the start: 2 copper layers, 27.5 x 14.5 mm, 13 parts, among them J1 Conn_01x04, J2 Conn_01x04, U1 LSM6DSM

Commit message: This is what was actually ordered.
Routing:
- net /SDA: track 27.4 -> 28.1 mm
- net GND: vias 3 -> 10
Changed lines of the file:
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@@
 		(tags "resistor")
 		(property "Reference" "R3"
-			(at 0 -1.43 360)
+			(at 0 -1.43 0)
 			(layer "F.SilkS")
 			(effects
@@
 		)
 		(property "Value" "330"
-			(at 0 1.43 360)
+			(at 0 1.43 0)
 			(layer "F.Fab")
 			(effects
@@
 		)
 		(fp_text user "${REFERENCE}"
-			(at 0 0 360)
+			(at 0 0 0)
 			(layer "F.Fab")
 			(effects
@@
 		(tags "LED")
 		(property "Reference" "D1"
-			(at 2.5 1 360)
+			(at 2.5 1 0)
 			(layer "F.SilkS")
 			(effects
@@
 		)
 		(property "Value" "LED"
-			(at 0 1.43 360)
+			(at 0 1.43 0)
 			(layer "F.Fab")
 			(effects
@@
 		)
 		(fp_text user "${REFERENCE}"
-			(at 0 0 360)
+			(at 0 0 0)
 			(layer "F.Fab")
 			(effects
@@
 		(tags "LGA NoLead")
 		(property "Reference" "U1"
-			(at 0 -2.2 360)
+			(at 0 -2.2 0)
 			(layer "F.SilkS")
 			(effects
@@
 		)
 		(property "Value" "LSM6DSM"
-			(at 0 2.2 360)
+			(at 0 2.2 0)
 			(layer "F.Fab")
 			(effects
@@
 		)
 		(fp_text user "${REFERENCE}"
-			(at 0 0 360)
+			(at 0 0 0)
 			(layer "F.Fab")
 			(effects
@@
 	)
 	(via
+		(at 165 104.5)
+		(size 0.8)
+		(drill 0.4)
+		(layers "F.Cu" "B.Cu")
+		(free yes)
+		(net 1)
+	)
+	(via
+		(at 164.5 101)
+		(size 0.8)
+		(drill 0.4)
+		(layers "F.Cu" "B.Cu")
+		(free yes)
+		(net 1)
+	)
+	(via
+		(at 148.25 94.25)
+		(size 0.8)
+		(drill 0.4)
+		(layers "F.Cu" "B.Cu")
+		(free yes)
+		(net 1)
+	)
+	(via
 		(at 159.618784 102.787638)
+		(size 0.8)
+		(drill 0.4)
+		(layers "F.Cu" "B.Cu")
+		(free yes)
+		(net 1)
+	)
+	(via
+		(at 170.25 96.25)
+		(size 0.8)
+		(drill 0.4)
+		(layers "F.Cu" "B.Cu")
+		(free yes)
+		(net 1)
+	)
+	(via
+		(at 161.75 99)
 		(size 0.8)
 		(drill 0.4)
@@
 		(net 1)
 	)
+	(via
+		(at 152.25 98)
+		(size 0.8)
+		(drill 0.4)
+		(layers "F.Cu" "B.Cu")
+		(free yes)
+		(net 1)
+	)
+	(via
+		(at 156.75 98.25)
+		(size 0.8)
+		(drill 0.4)
+		(layers "F.Cu" "B.Cu")
+		(free yes)
+		(net 1)
+	)
 	(segment
 		(start 164.2 96.7)
@@
 	)
 	(segment
+		(start 156 99.75)
+		(end 156 99.24)
+		(width 0.127)
+		(layer "B.Cu")
+		(net 4)
+	)
+	(segment
+		(start 167.8 99.24)
+		(end 167.29 99.75)
+		(width 0.127)
+		(layer "B.Cu")
+		(net 4)
+	)
+	(segment
+		(start 167.29 99.75)
+		(end 156 99.75)
+		(width 0.127)
+		(layer "B.Cu")
+		(net 4)
+	)
+	(segment
 		(start 150.08 100)
 		(end 148.3 101.78)
@@
 		(start 153.26 99.24)
 		(end 152.5 100)
-		(width 0.1524)
-		(layer "B.Cu")
-		(net 4)
-	)
-	(segment
-		(start 167.8 99.24)
-		(end 156 99.24)
 		(width 0.1524)
 		(layer "B.Cu")
@@
 		(hatch edge 0.5)
 		(connect_pads
-			(clearance 0.5)
-		)
-		(min_thickness 0.25)
+			(clearance 0.2)
+		)
+		(min_thickness 0.2)
 		(filled_areas_thickness no)
 		(fill yes
@@
 		(hatch edge 0.5)
 		(connect_pads
-			(clearance 0.5)
-		)
-		(min_thickness 0.25)
+			(clearance 0.2)
+		)
+		(min_thickness 0.2)
 		(filled_areas_thickness no)
 		(fill yes
