File: electronics/STImu.kicad_sch (KiCad schematic)
At the start: 13 parts, among them J1 Conn_01x04, J2 Conn_01x04, U1 LSM6DSM

Commit message: This is what was actually ordered.
Parts:
- R5: now not fitted
